File: _autosave-Stopwatch_Timer.kicad_pcb (KiCad board)
At the start: 2 copper layers, 250 x 200 mm, 89 parts, among them J1 Conn_01x02_Socket, J2 Conn_01x03_Socket, SW1 SW_DIP_x08, SW2 SW_DIP_x04, SW3 SW_DIP_x08, U1 NE555P, U10 74LS157, U11 SN74HC04N, U12 CD4075BE, U13 SN74HC04N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

Commit message: Testing the CADLAB
Parts:
- moved U18 132.0 mm to (95.3, 41.6)
- moved R11 18.5 mm to (280.8, -131.3)
- moved R21 18.5 mm to (294.1, -131.3)
- moved C1 18.5 mm to (36.8, 184.1)
- moved C2 18.5 mm to (49.7, 170.2)
- moved J1 18.5 mm to (22.9, 175.3)
- moved J2 18.5 mm to (310.4, -98.5)
- moved MT1 18.5 mm to (175.6, -91.7)
- moved MU1 18.5 mm to (186.4, -91.7)
- moved R10 18.5 mm to (175.6, -37.4)
- moved R12 18.5 mm to (280.8, -127.2)
- moved R13 18.5 mm to (280.8, -123.2)
- moved R14 18.5 mm to (280.8, -119.1)
- moved R15 18.5 mm to (280.8, -115.1)
- moved R16 18.5 mm to (280.8, -111.0)
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
Commit message: Second Test
Parts:
- moved U18 7.60 mm to (102.5, 44.1)
Changed lines of the file:
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@@
 	(footprint "Package_DIP:DIP-14_W7.62mm_Socket"
 		(layer "F.Cu")
-		(at 95.3 41.63 -90)
+		(at 102.48 44.13 -90)
 		(descr "14-lead though-hole mounted DIP package, row spacing 7.62mm (300 mils), Socket")
 		(tags "THT DIP DIL PDIP 2.54mm 7.62mm 300mil Socket")
