File: Stopwatch_Timer.kicad_sch (KiCad schematic)
At the start: 93 parts, among them J1 Conn_01x02_Socket, J2 Conn_01x03_Socket, SW1 SW_DIP_x08, SW2 SW_DIP_x04, SW3 SW_DIP_x08, U1 NE555P, U10 74LS157, U11 SN74HC04N, U12 CD4075BE, U13 SN74HC04N, U14 HDSP-A151, U15 HDSP-A151, U16 HDSP-A151, U17 HDSP-A151, U18 SN74HC32N, U19 SN74HC08N, U20 SN74HC32N, U21 CD4075BE, U22 CD4023BE, U23 SN74HC32N, U24 SN74HC08N, U4 74LS47, U6 74LS47, U7 74LS47, U9 74LS47

Commit message: Done part of the routing
Parts:
- removed U14, U15, U16, U17: HDSP-A151, Display_7Segment:7SegmentLED_LTS6760_LTS6780, symbol Display_Character:HDSP-A151
- S3: value BUTT-2 -> Set_Button
- S4: value BUTT-2 -> Global_Reset
- S5: value BUTT-2 -> Start/Pause
- renumbered U6 to MT2, AFF1 to MT3, U4 to MU2, AFF2 to MU3, R4 to RMT_1, R5 to RMT_2, R6 to RMT_3, R7 to RMT_4, R8 to RMT_5, R9 to RMT_6, R10 to RMT_7, R11 to RMU_1, R12 to RMU_2, R13 to RMU_3, R14 to RMU_4, R15 to RMU_5, R16 to RMU_6, R17 to RMU_7, R18 to RST_1, R19 to RST_2, R20 to RST_3, R21 to RST_4, R22 to RST_5, R23 to RST_6, R24 to RST_7, R25 to RSU_1, R26 to RSU_2, R27 to RSU_3, R28 to RSU_4, R29 to RSU_5, R30 to RSU_6, R31 to RSU_7, R40 to R_SW_MT_1, R41 to R_SW_MT_2, R42 to R_SW_MT_3, R43 to R_SW_MT_4, R44 to R_SW_MU_1, R45 to R_SW_MU_2, R46 to R_SW_MU_3, R47 to R_SW_MU_4, R3 to R_SW_ST_1, R32 to R_SW_ST_2, R33 to R_SW_ST_3, R34 to R_SW_ST_4, R35 to R_SW_SU_1, R36 to R_SW_SU_2, R37 to R_SW_SU_3, R38 to R_SW_SU_4, U7 to ST2, AFF3 to ST3, U9 to SU2, AFF4 to SU3, SW3 to SW_M1, SW1 to SW_S1
Connections:
- net +5V: now also MT3.3 (C.A.), MT3.5 (DP), MT3.8 (C.A.), MU3.3 (C.A.), MU3.5 (DP), MU3.8 (C.A.), ST3.3 (C.A.), ST3.5 (DP), ST3.8 (C.A.), SU3.3 (C.A.), SU3.5 (DP), SU3.8 (C.A.)
- net at RMU_1.2: now also MU3.7 (a)
- net at RMT_3.2: now also MT3.4 (c)
- net at RMU_5.2: now also MU3.1 (e)
- net at RST_2.2: now also ST3.6 (b)
- net at RMU_2.2: now also MU3.6 (b)
- net at RMT_2.2: now also MT3.6 (b)
- net at RMU_4.2: now also MU3.2 (d)
- net at SU3.1 (e): now also RSU_5.2
- net at SU3.10 (g): now also RSU_7.2
- net at SU3.2 (d): now also RSU_4.2
- net at SU3.4 (c): now also RSU_3.2
- net at SU3.6 (b): now also RSU_2.2
- net at SU3.7 (a): now also RSU_1.2
- net at SU3.9 (f): now also RSU_6.2
- net at RMT_1.2: now also MT3.7 (a)
- net at RMT_5.2: now also MT3.1 (e)
- net at ST3.1 (e): now also RST_5.2
- net at ST3.10 (g): now also RST_7.2
- net at ST3.2 (d): now also RST_4.2
- net at ST3.4 (c): now also RST_3.2
- net at ST3.7 (a): now also RST_1.2
- net at ST3.9 (f): now also RST_6.2
- net at MT3.10 (g): now also RMT_7.2
- net at MT3.2 (d): now also RMT_4.2
- net at MT3.9 (f): now also RMT_6.2
- net at RMU_6.2: now also MU3.9 (f)
- net at MU3.10 (g): now also RMU_7.2
- net at MU3.4 (c): now also RMU_3.2
Other:
- moved on the sheet: MT3, MU3, ST3, SU3

Commit message: Final PCB design
Parts:
- S3: value Set_Button -> BUTT-2
- S4: value Global_Reset -> BUTT-2
- S5: value Start/Pause -> BUTT-2
- renumbered MT3 to AFF1, MU3 to AFF2, ST3 to AFF3, SU3 to AFF4, RMT_7 to R10, RMU_1 to R11, RMU_2 to R12, RMU_3 to R13, RMU_4 to R14, RMU_5 to R15, RMU_6 to R16, RMU_7 to R17, RST_1 to R18, RST_2 to R19, RST_3 to R20, RST_4 to R21, RST_5 to R22, RST_6 to R23, RST_7 to R24, RSU_1 to R25, RSU_2 to R26, RSU_3 to R27, RSU_4 to R28, RSU_5 to R29, R_SW_ST_1 to R3, RSU_6 to R30, RSU_7 to R31, R_SW_ST_2 to R32, R_SW_ST_3 to R33, R_SW_ST_4 to R34, R_SW_SU_1 to R35, R_SW_SU_2 to R36, R_SW_SU_3 to R37, R_SW_SU_4 to R38, RMT_1 to R4, R_SW_MT_1 to R40, R_SW_MT_2 to R41, R_SW_MT_3 to R42, R_SW_MT_4 to R43, R_SW_MU_1 to R44, R_SW_MU_2 to R45, R_SW_MU_3 to R46, R_SW_MU_4 to R47, RMT_2 to R5, RMT_3 to R6, RMT_4 to R7, RMT_5 to R8, RMT_6 to R9, SW_S1 to SW1, SW_M1 to SW3, MU2 to U4, MT2 to U6, ST2 to U7, SU2 to U9
Other:
- moved on the sheet: AFF1, AFF2, AFF3, AFF4

Commit message: Finalized PCB design
Parts:
- removed J1: Conn_01x02_Socket, Connector_PinSocket_2.54mm:PinSocket_1x02_P2.54mm_Vertical, symbol Connector:Conn_01x02_Socket
- removed J2: Conn_01x03_Socket, Connector_PinSocket_2.54mm:PinSocket_1x03_P2.54mm_Vertical, symbol Connector:Conn_01x03_Socket
- added J3: Conn_01x06_Socket, Connector_PinSocket_2.54mm:PinSocket_1x06_P2.54mm_Vertical, symbol Connector:Conn_01x06_Socket
Connections:
- net +5V: now also J3.1 (Pin_1), J3.4 (Pin_4)
- net GND: now also J3.2 (Pin_2), J3.6 (Pin_6)
- net at R46.1, SW3.10: now also MU1.1 (B); no longer MU1.10 (C)
- net at R45.1, SW3.11: now also MU1.10 (C); no longer MU1.1 (B)
- net at R44.1, SW3.12: now also MU1.9 (D); no longer MU1.15 (A)
- net at R43.1, SW3.13: now also MT1.15 (A); no longer MT1.9 (D)
- net at R42.1, SW3.14: now also MT1.1 (B); no longer MT1.10 (C)
- net at R41.1, SW3.15: now also MT1.10 (C); no longer MT1.1 (B)
- net at R40.1, SW3.16: now also MT1.9 (D); no longer MT1.15 (A)
- net at R47.1, SW3.9: now also MU1.15 (A); no longer MU1.9 (D)
- net at U13.13 (6A), U18.8 (3Y): now also J3.5 (Pin_5)
