File: Stopwatch_Timer.kicad_pcb (KiCad board)
At the start: 2 copper layers, 250 x 200 mm, 89 parts, among them J1 Conn_01x02_Socket, J2 Conn_01x03_Socket, SW1 SW_DIP_x08, SW2 SW_DIP_x04, SW3 SW_DIP_x08, U1 NE555P, U10 74LS157, U11 SN74HC04N, U12 CD4075BE, U13 SN74HC04N, U14 HDSP-A151, U15 HDSP-A151, U16 HDSP-A151, U17 HDSP-A151, U18 SN74HC32N, U19 SN74HC08N, U20 SN74HC32N, U21 CD4075BE, U22 CD4023BE, U23 SN74HC32N, U24 SN74HC08N, U4 74LS47, U6 74LS47, U7 74LS47, U9 74LS47

Commit message: Test parallel work
Parts:
- moved R33 437.3 mm to (-92.4, 1.24)
- moved R34 437.3 mm to (-92.4, 5.24)
- moved R35 349.8 mm to (98.5, 122.8)
- moved R36 349.8 mm to (98.5, 126.8)
- moved R37 349.8 mm to (98.5, 130.8)
- moved R38 349.8 mm to (98.5, 134.8)
- moved S4 348.7 mm to (65.7, 141.1)
- moved R3 322.6 mm to (-92.4, -6.76)
- moved R32 322.6 mm to (-92.4, -2.76)
- moved R29 285.3 mm to (512.7, 57.4), turned to 90 degrees
- moved R28 284.3 mm to (508.7, 57.4), turned to 90 degrees
- moved R27 283.4 mm to (504.7, 57.4), turned to 90 degrees
- moved R26 282.6 mm to (500.7, 57.4), turned to 90 degrees
- moved R25 281.9 mm to (496.7, 57.4), turned to 90 degrees
- moved R31 279.4 mm to (492.7, 57.4), turned to 90 degrees
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Connections:
- R35 pad 1: Net-(SU1-A) -> Net-(SU1-D)
- R36 pad 1: Net-(SU1-B) -> Net-(SU1-C)
- R37 pad 1: Net-(SU1-C) -> Net-(SU1-B)
- R38 pad 1: Net-(SU1-D) -> Net-(SU1-A)
- SW1 pad 10: Net-(SU1-C) -> Net-(SU1-B)
- SW1 pad 11: Net-(SU1-B) -> Net-(SU1-C)
- SW1 pad 12: Net-(SU1-A) -> Net-(SU1-D)
- SW1 pad 9: Net-(SU1-D) -> Net-(SU1-A)
Routing:
- net +5V: track 145.3 -> 192.6 mm
- net GND: track 117.7 -> 147.0 mm, vias 0 -> 1
- net Net-(U20-3A): track 0.00 -> 13.5 mm
- net Net-(U13-1Y): track 37.1 -> 34.7 mm
- net Net-(U20-1A): track 36.1 -> 36.9 mm

Commit message: Done part of the routing
Parts:
- removed U14, U15, U16, U17: HDSP-A151, Display_7Segment:7SegmentLED_LTS6760_LTS6780
- added MT3: LTS-6960HR, Display_7Segment:7SegmentLED_LTS6760_LTS6780, F.Cu at (196.6, 28.6)
- added MU3: LTS-6960HR, Display_7Segment:7SegmentLED_LTS6760_LTS6780, F.Cu at (213.7, 28.5)
- added ST3: LTS-6960HR, Display_7Segment:7SegmentLED_LTS6760_LTS6780, F.Cu at (230.7, 28.5)
- added SU3: LTS-6960HR, Display_7Segment:7SegmentLED_LTS6760_LTS6780, F.Cu at (247.3, 28.6)
- S3: value BUTT-2 -> Set_Button
- S4: value BUTT-2 -> Global_Reset
- S5: value BUTT-2 -> Start/Pause
- moved R_SW_ST_4 360.0 mm to (221.6, 181.2)
- moved R50 359.0 mm to (154.6, 193.3), turned to 90 degrees
- moved R_SW_ST_3 358.9 mm to (221.6, 175.0)
- moved R_SW_ST_2 358.0 mm to (221.6, 169.3)
- moved R_SW_ST_1 357.0 mm to (221.5, 163.2)
- moved S3 355.2 mm to (153.6, 177.5)
- moved SW_M1 339.1 mm to (185.5, 196.0), turned to 90 degrees
- moved U11 320.7 mm to (152.2, 135.4)
- moved R_SW_MU_4 309.5 mm to (201.6, 181.1)
- moved R_SW_MU_3 308.2 mm to (201.6, 174.9)
- moved R_SW_MU_2 307.1 mm to (201.6, 169.2)
- moved R_SW_MU_1 306.0 mm to (201.7, 163.2)
- moved R_SW_MT_4 301.6 mm to (178.3, 181.1)
- moved R_SW_MT_3 300.2 mm to (178.3, 174.9)
- moved R_SW_MT_2 299.0 mm to (178.3, 169.2)
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- renumbered U6 to MT2, U4 to MU2, R4 to RMT_1, R5 to RMT_2, R6 to RMT_3, R7 to RMT_4, R8 to RMT_5, R9 to RMT_6, R10 to RMT_7, R11 to RMU_1, R12 to RMU_2, R13 to RMU_3, R14 to RMU_4, R15 to RMU_5, R16 to RMU_6, R17 to RMU_7, R18 to RST_1, R19 to RST_2, R20 to RST_3, R21 to RST_4, R22 to RST_5, R23 to RST_6, R24 to RST_7, R25 to RSU_1, R26 to RSU_2, R27 to RSU_3, R28 to RSU_4, R29 to RSU_5, R30 to RSU_6, R31 to RSU_7, R40 to R_SW_MT_1, R41 to R_SW_MT_2, R42 to R_SW_MT_3, R43 to R_SW_MT_4, R44 to R_SW_MU_1, R45 to R_SW_MU_2, R46 to R_SW_MU_3, R47 to R_SW_MU_4, R3 to R_SW_ST_1, R32 to R_SW_ST_2, R33 to R_SW_ST_3, R34 to R_SW_ST_4, R35 to R_SW_SU_1, R36 to R_SW_SU_2, R37 to R_SW_SU_3, R38 to R_SW_SU_4, U7 to ST2, U9 to SU2, SW3 to SW_M1, SW1 to SW_S1
Routing:
- net +5V: track 192.6 -> 1284.2 mm, vias 7 -> 5
- net GND: track 147.0 -> 1059.9 mm, vias 1 -> 4
- net Net-(MT1-~{LOAD}): track 0.00 -> 455.2 mm, vias 0 -> 3
- net Net-(ST1-QC): track 0.00 -> 361.0 mm, vias 0 -> 4
- net Net-(ST1-QB): track 0.00 -> 302.9 mm, vias 0 -> 3
- net Net-(ST1-QA): track 0.00 -> 293.5 mm, vias 0 -> 3
- net Net-(MT1-CLR): track 0.00 -> 293.4 mm, vias 0 -> 3
- net Net-(U10-I0a): track 0.00 -> 291.0 mm, vias 0 -> 1
- net Net-(ST1-QD): track 0.00 -> 268.9 mm, vias 0 -> 3
- net Net-(U11-3Y): track 0.00 -> 255.8 mm, vias 0 -> 1
- net Net-(MU1-DOWN): track 0.00 -> 233.8 mm, vias 0 -> 3
- net Net-(U10-I0b): track 0.00 -> 224.0 mm, vias 0 -> 1
- net Net-(U11-3A): track 50.6 -> 269.7 mm, vias 0 -> 2
- net Net-(U10-I0d): track 0.00 -> 215.2 mm, vias 0 -> 1
- net Net-(U10-I0c): track 0.00 -> 215.1 mm, vias 0 -> 1
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Other:
- board text removed: "${REFERENCE}"

Commit message: Final PCB design
Parts:
- removed MT3, MU3, ST3, SU3: LTS-6960HR, Display_7Segment:7SegmentLED_LTS6760_LTS6780
- added AFF1: LTS-6960HR, Display_7Segment:7SegmentLED_LTS6760_LTS6780, F.Cu at (248.0, 75.7)
- added AFF2: LTS-6960HR, Display_7Segment:7SegmentLED_LTS6760_LTS6780, F.Cu at (247.8, 97.4)
- added AFF3: LTS-6960HR, Display_7Segment:7SegmentLED_LTS6760_LTS6780, F.Cu at (247.9, 120.1)
- added AFF4: LTS-6960HR, Display_7Segment:7SegmentLED_LTS6760_LTS6780, F.Cu at (247.8, 141.8)
- S3: value Set_Button -> BUTT-2
- S4: value Global_Reset -> BUTT-2
- S5: value Start/Pause -> BUTT-2
- moved SW3 212.7 mm to (25.0, 56.4), turned to 0 degrees
- moved SW1 205.0 mm to (48.6, 102.0), turned to 0 degrees
- moved R38 189.3 mm to (66.6, 128.0)
- moved R37 188.6 mm to (66.6, 124.0)
- moved R36 188.0 mm to (66.6, 120.0)
- moved R35 187.3 mm to (66.6, 116.0)
- moved R47 184.9 mm to (44.0, 84.4)
- moved R46 183.8 mm to (44.0, 80.4)
- moved R45 182.9 mm to (44.0, 76.4)
- moved R44 182.0 mm to (44.0, 72.4)
- moved R43 175.3 mm to (44.0, 68.4)
- moved R42 174.0 mm to (44.0, 64.4)
- moved R41 172.8 mm to (44.0, 60.4)
- moved R40 171.6 mm to (44.0, 56.4)
- moved U19 170.4 mm to (171.4, 192.6)
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- renumbered RMT_7 to R10, RMU_1 to R11, RMU_2 to R12, RMU_3 to R13, RMU_4 to R14, RMU_5 to R15, RMU_6 to R16, RMU_7 to R17, RST_1 to R18, RST_2 to R19, RST_3 to R20, RST_4 to R21, RST_5 to R22, RST_6 to R23, RST_7 to R24, RSU_1 to R25, RSU_2 to R26, RSU_3 to R27, RSU_4 to R28, RSU_5 to R29, R_SW_ST_1 to R3, RSU_6 to R30, RSU_7 to R31, R_SW_ST_2 to R32, R_SW_ST_3 to R33, R_SW_ST_4 to R34, R_SW_SU_1 to R35, R_SW_SU_2 to R36, R_SW_SU_3 to R37, R_SW_SU_4 to R38, RMT_1 to R4, R_SW_MT_1 to R40, R_SW_MT_2 to R41, R_SW_MT_3 to R42, R_SW_MT_4 to R43, R_SW_MU_1 to R44, R_SW_MU_2 to R45, R_SW_MU_3 to R46, R_SW_MU_4 to R47, RMT_2 to R5, RMT_3 to R6, RMT_4 to R7, RMT_5 to R8, RMT_6 to R9, SW_S1 to SW1, SW_M1 to SW3, MU2 to U4, MT2 to U6, ST2 to U7, SU2 to U9
Routing:
- net Net-(U10-I0a): track 291.0 -> 61.8 mm, vias 1 -> 0
- net Net-(U11-3Y): track 255.8 -> 54.2 mm, vias 1 -> 3
- net Net-(MT1-~{LOAD}): track 455.2 -> 258.2 mm, vias 3 -> 2
- net Net-(MU1-DOWN): track 233.8 -> 37.1 mm, vias 3 -> 0
- net Net-(ST1-QC): track 361.0 -> 178.1 mm, vias 4 -> 0
- net Net-(U10-I0b): track 224.0 -> 56.7 mm
- net Net-(ST1-~{LOAD}): track 199.2 -> 48.2 mm
- net Net-(U10-I0c): track 215.1 -> 70.9 mm, vias 1 -> 0
- net Net-(U10-I0d): track 215.2 -> 71.7 mm, vias 1 -> 0
- net Net-(ST1-QB): track 302.9 -> 169.8 mm, vias 3 -> 0
- net Net-(SU1-UP): track 203.1 -> 72.9 mm
- net Net-(SU1-DOWN): track 193.4 -> 65.3 mm
- net Net-(U11-1A): track 189.4 -> 70.4 mm
- net Net-(ST1-QD): track 268.9 -> 175.0 mm, vias 3 -> 2
- net Net-(U11-3A): track 269.7 -> 179.6 mm, vias 2 -> 1
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Other:
- board size 250 x 200 mm -> 278.6 x 218.9 mm

Commit message: Finalized PCB design
Parts:
- removed J1: Conn_01x02_Socket, Connector_PinSocket_2.54mm:PinSocket_1x02_P2.54mm_Vertical
- removed J2: Conn_01x03_Socket, Connector_PinSocket_2.54mm:PinSocket_1x03_P2.54mm_Vertical
- added J3: Conn_01x06_Socket, Connector_PinSocket_2.54mm:PinSocket_1x06_P2.54mm_Vertical, F.Cu at (61.4, 180.2)
- moved S3 93.4 mm to (48.4, 149.8)
- moved SW2 78.4 mm to (26.1, 120.7), turned to 0 degrees
- moved U18 62.5 mm to (107.3, 76.6)
- moved R1 57.2 mm to (73.9, 166.4)
- moved R34 51.5 mm to (55.5, 105.3), turned to 0 degrees
- moved R33 48.8 mm to (55.5, 100.8), turned to 0 degrees
- moved R32 46.7 mm to (55.5, 96.2), turned to 0 degrees
- moved R39 46.0 mm to (66.4, 155.9)
- moved R3 45.4 mm to (55.5, 91.6), turned to 0 degrees
- moved U20 36.6 mm to (92.0, 163.8)
- moved S5 35.1 mm to (48.3, 163.8), turned to 0 degrees
- moved R_Mode1 31.9 mm to (74.0, 145.6), turned to 180 degrees
- moved C1 26.8 mm to (50.9, 175.3), turned to -90 degrees
- moved SW1 24.9 mm to (26.0, 91.6)
- moved U21 21.7 mm to (107.3, 51.6)
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Connections:
- R40 pad 1: Net-(MT1-A) -> Net-(MT1-D)
- R41 pad 1: Net-(MT1-B) -> Net-(MT1-C)
- R42 pad 1: Net-(MT1-C) -> Net-(MT1-B)
- R43 pad 1: Net-(MT1-D) -> Net-(MT1-A)
- R44 pad 1: Net-(MU1-A) -> Net-(MU1-D)
- R45 pad 1: Net-(MU1-B) -> Net-(MU1-C)
- R46 pad 1: Net-(MU1-C) -> Net-(MU1-B)
- R47 pad 1: Net-(MU1-D) -> Net-(MU1-A)
- SW3 pad 10: Net-(MU1-C) -> Net-(MU1-B)
- SW3 pad 11: Net-(MU1-B) -> Net-(MU1-C)
- SW3 pad 12: Net-(MU1-A) -> Net-(MU1-D)
- SW3 pad 13: Net-(MT1-D) -> Net-(MT1-A)
- SW3 pad 14: Net-(MT1-C) -> Net-(MT1-B)
- SW3 pad 15: Net-(MT1-B) -> Net-(MT1-C)
- SW3 pad 16: Net-(MT1-A) -> Net-(MT1-D)
- SW3 pad 9: Net-(MU1-D) -> Net-(MU1-A)
Routing:
- net +5V: track 1248.4 -> 1067.9 mm, vias 3 -> 2
- net GND: track 1004.8 -> 850.2 mm, vias 0 -> 2
- net Net-(J3-Pin_5): track 211.2 -> 123.1 mm
- net Net-(U19-2Y): track 156.4 -> 86.2 mm
- net Net-(U1-OUT): track 6.26 -> 60.4 mm, vias 0 -> 1
- net Net-(MT1-CLR): track 217.1 -> 163.2 mm
- net Net-(U18-2A): track 71.0 -> 18.3 mm, vias 2 -> 0
- net Net-(U11-3A): track 179.6 -> 229.9 mm
- net Net-(U18-1A): track 87.0 -> 36.6 mm
- net Net-(U20-3A): track 24.1 -> 68.6 mm, vias 0 -> 1
- net Net-(U18-1B): track 72.3 -> 29.1 mm, vias 1 -> 0
- net Net-(SU1-C): track 104.0 -> 145.6 mm
- net Net-(MU1-UP): track 71.5 -> 112.9 mm, vias 1 -> 3
- net Net-(MU1-QD): track 162.4 -> 121.4 mm, vias 1 -> 0
- net Net-(U11-2A): track 143.2 -> 102.5 mm
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Other:
- board size 278.6 x 218.9 mm -> 245.6 x 138.6 mm
- board text added: "555 timer"
- board text added: "61-33960 61-37001 61-29627 61-14444 61-34156"
- board text added: "7-segment MT"
- board text added: "7-segment MU"
- board text added: "7-segment ST"
- board text added: "7-segment SU"
- board text added: "All Hail King Dr.AbdelGhany !!"
- board text added: "Button"
- board text added: "C 10nF"
- board text added: "C 10uF"
- board text added: "CD4023 3-input NAND"
- board text added: "CD4075 3-input OR"
- board text added: "ELCT Class 2028"
- board text added: "GND"
- board text added: "IN"
- board text added: "Minutes_IN"
- board text added: "Morkos Shenouda Youssef Tarek ABDO FARAG Ahmed Diaa Muhammad Walid"
- board text added: "Pause"
- board text added: "Power"
- board text added: "Push"
- board text added: "R 10k"
- board text added: "R 1k"
- board text added: "R 22k"
- board text added: "R 330"
- board text added: "Relay Pins"
- board text added: "Reset"
- board text added: "SN74HC04N NOT"
- board text added: "SN74HC08N 2-input AND"
- board text added: "SN74HC32N 2-input OR"
- board text added: "SN74LS157N MUX"
- board text added: "SN74LS192N counter MT"
- board text added: "SN74LS192N counter MU"
- board text added: "SN74LS192N counter ST"
- board text added: "SN74LS192N counter SU"
- board text added: "SN74LS47N 7-segment decoder"
- board text added: "Seconds_IN"
- board text added: "Set"
- board text added: "UP/DOWN"
- board text added: "VCC"

Commit message: replaced silkscreen text with copper text
Routing:
- net Net-(AFF1-f): track 58.0 -> 47.5 mm
- net Net-(U1-OUT): track 60.4 -> 56.1 mm
- net Net-(U11-3A): track 229.9 -> 232.6 mm
Other:
- board text added: "All Hail King Dr. AbdelGhany !!"
- board text removed: "555 timer"
- board text removed: "7-segment MT"
- board text removed: "7-segment MU"
- board text removed: "7-segment ST"
- board text removed: "7-segment SU"
- board text removed: "All Hail King Dr.AbdelGhany !!"
- board text removed: "Button"
- board text removed: "C 10nF"
- board text removed: "C 10uF"
- board text removed: "CD4023 3-input NAND"
- board text removed: "CD4075 3-input OR"
- board text removed: "GND"
- board text removed: "IN"
- board text removed: "Power"
- board text removed: "Push"
- board text removed: "R 10k"
- board text removed: "R 1k"
- board text removed: "R 22k"
- board text removed: "R 330"
- board text removed: "Relay Pins"
- board text removed: "SN74HC04N NOT"
- board text removed: "SN74HC08N 2-input AND"
- board text removed: "SN74HC32N 2-input OR"
- board text removed: "SN74LS157N MUX"
- board text removed: "SN74LS192N counter MT"
- board text removed: "SN74LS192N counter MU"
- board text removed: "SN74LS192N counter ST"
- board text removed: "SN74LS192N counter SU"
- board text removed: "SN74LS47N 7-segment decoder"
- board text removed: "VCC"
